File: Board_UV V 0.1.sch (EAGLE design)
At the start: 32 parts, among them IC4 74HC14D, IC5 MAX3232CSE, U1 TLP521-4(GB), U2 TLP521-4(GB), U3 TLP521-4(GB)

Commit message: Add other component
Parts:
- added JP1, JP2: (no value), pinhead:PINHD-1X8
- added JP3: (no value), pinhead:PINHD-1X2
- added JP4: (no value), pinhead:PINHD-1X16
- added JP5: (no value), pinhead:PINHD-1X4
- added JP6: (no value), pinhead:PINHD-1X6
- added JP7: (no value), pinhead:PINHD-1X12
- added JP8: (no value), pinhead:PINHD-1X3
- added LS1: BUZZER-PTH_KIT, SparkFun-Electromechanical:BUZZER-PTH_KIT
- added Q1, Q2: 500mA/300V, SparkFun-DiscreteSemi:TRANS_NPN-MMBTA42
- added R21, R22: 2k2, SparkFun-Resistors:10KOHM-0603-1/10W-1%
- added R23, R25, R26, R27, R28, R29: 1k, SparkFun-Resistors:10KOHM-0603-1/10W-1%
- added R24: 10k, SparkFun-Resistors:10KOHM-0603-1/10W-1%
- added R30, R31, R32, R33, R34, R35: 330, SparkFun-Resistors:10KOHM-0603-1/10W-1%
Connections:
- new net 1A: JP2.4
- new net 1B: JP2.3
- new net 2A: JP2.5
- new net 2B: JP2.6
- new net BTN-1: U$1.A14
- new net BTN-2: U$1.D32
- new net BTN-3: U$1.D34
- new net BTN-4: U$1.D36
- new net BTN-5: U$1.D38
- new net BUZ-12V: U$1.D13
- new net BUZ-5V: U$1.D11
- new net DHT: U$1.D7
- new net DIR: JP1.8, U$1.D45
- new net EN: JP1.1, U$1.D43
- new net LCD-D11: U$1.A8
- new net LCD-D12: U$1.A10
- new net LCD-D2: U$1.A0
- new net LCD-D3: U$1.A2
- new net LCD-D4: U$1.A4
- new net LCD-D5: U$1.A6
- new net LED-1: U$1.D40
- new net LED-2: U$1.D42
- new net LED-3: U$1.D44
- new net LED-4: U$1.D46
- new net LED-5: U$1.D48
- new net LIM-B1: U$1.D22
- new net LIM-B2: U$1.D24
- new net LIM-B3: U$1.D26
- new net LIM-B4: U$1.D28
- new net LIM-CTR: U$1.D21
- new net LIM-S1: U$1.D30
- new net LIM-S2: U$1.D31
- new net MISO: JP1.2, U$1.D50
- new net MOSI: JP1.5, U$1.D51
- new net N$101: JP8.3
- new net N$25: Q1.B, R21.1
- new net N$41: R21.2, R22.2
- new net N$42: LS1.2, Q1.C
- new net N$66: Q2.B, R22.1
- new net N$67: JP3.2
- new net N$68: Q2.C
- new net N$69: R24.2, U2.A3
- new net N$70: JP6.6, R25.1
- new net N$71: JP4.3, R23.1
- new net N$72: JP4.4
- new net N$73: JP5.2
- new net N$74: JP4.6
- new net N$75: JP5.3
- new net N$76: JP6.5, R26.1
- new net N$77: JP4.14
- new net N$78: JP4.13
- new net N$79: JP4.12
- new net N$80: JP4.11
- new net N$81: JP6.4, R27.1
- new net N$82: JP6.3, R28.1
- new net N$83: JP6.2, R29.1
- new net N$84: U2.CT3
- new net N$85: JP7.7, R33.2
- new net N$86: R24.1
- new net N$87: JP7.1, R30.2
- new net N$88: JP7.2
- new net N$89: JP7.3, R31.2
- new net N$90: JP7.4
- new net N$91: JP7.5, R32.2
- new net N$92: JP7.6
- new net N$93: JP7.8
- new net N$94: JP7.9, R34.2
- new net N$95: JP7.10
- new net N$96: JP7.11, R35.2
- new net N$97: JP7.12
- new net RL-1: U$1.D23
- new net RL-2: U$1.D25
- new net RL-3: U$1.D27
- new net RL-4: U$1.D29
- new net RX-DB9: U$1.D17
- new net RX-PWR: U$1.D19
- new net SCK: JP1.3, U$1.D52
- new net SPDT-1: U$1.D33
- new net SPDT-2: U$1.D35
- new net SPDT-3: U$1.D37
- new net SPDT-4: U$1.D39
- new net SPDT-5: U$1.D41
- new net SS: JP1.4, U$1.D53
- new net STEP: JP1.7, U$1.D49
- new net TX-DB9: U$1.D16
- new net TX-PWR: U$1.D18
- net GND: now also JP2.1, JP4.1, JP4.16, JP4.5, JP5.4, JP8.1, Q1.E, Q2.E, R25.2, R26.2, R27.2, R28.2, R29.2, U$1.GND.1, U$1.GND.2, U2.ET3
- net GND-ISO: now also JP2.7, U2.C3
- net VCC: now also JP2.2, JP4.15, JP4.2, JP5.1, JP6.1, JP8.2, LS1.1, R23.2, R30.1, R31.1, R32.1, R33.1, R34.1, R35.1, U$1.+5V.1, U$1.+5V.2, U$1.VIN.1, U$1.VIN.2
- net VCC_2: now also JP2.8, JP3.1
Other:
- moved on the sheet: C1, C2, C3, C4, C5, IC4A, IC4B, IC4C, IC4D, IC4E, IC4F, IC4P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

Commit message: add board design
Parts:
- removed JP3: (no value), pinhead:PINHD-1X2
- removed JP4: (no value), pinhead:PINHD-1X16
- removed JP5: (no value), pinhead:PINHD-1X4
- removed JP6: (no value), pinhead:PINHD-1X6
- removed JP7: (no value), pinhead:PINHD-1X12
- removed JP8: (no value), pinhead:PINHD-1X3
- added DS1: LCM-S02004DSF, LCM-S02004DSF:LCM-S02004DSF
- added H1, H2, H3, H4: MOUNT-PAD-SQUARE3.0, holes:MOUNT-PAD-SQUARE3.0
- added IC1: 74HC14D, 74xx-eu:74HC14D
- added J2: POWER_JACK, SparkFun-Connectors:POWER_JACK
- added LED1, LED2, LED3, LED4, LED5, LED6: (no value), led:LED5MM
- added R36, R37, R38, R39, R41, R42: 1k, SparkFun-Resistors:10KOHM-0603-1/10W-1%
- added S1, S2, S3, S4, S5: MOMENTARY-SWITCH-SPST-PTH-12MM, SparkFun-Switches:MOMENTARY-SWITCH-SPST-PTH-12MM
- added U$2, U$3, U$4, U$5, U$6, U$7: ROCKER, rocker sw:ROCKER
- added U$8: DC-DC-STEP-DOWN-LM2596, diy-modules:DC-DC-STEP-DOWN-LM2596
- added X1: 22-23-2021, con-molex:22-23-2021
- added X2: 1751303, con-phoenix-350:1751303
- added X3: 1751277, con-phoenix-350:1751277
- added X4: 22-23-2031, con-molex:22-23-2031
- added X5: 22-23-2041, con-molex:22-23-2041
- added X6: 1751280, con-phoenix-350:1751280
- R23: value 1k -> 10k
Connections:
- removed net N$101: JP8.3
- removed net N$11: R1.2
- removed net N$12: IC4D.I, R2.2, U1.CT1
- removed net N$17: IC4E.I, R3.2, U1.CT2
- removed net N$18: IC4F.I, R5.1, U1.CT3
- removed net N$19: IC4A.I, R6.1, U1.CT4
- removed net N$20: R4.1
- removed net N$21: R7.1
- removed net N$22: R8.1
- removed net N$26: R9.2
- removed net N$27: IC4B.I, R10.2, U2.CT1
- removed net N$28: IC4C.I, R11.2, U2.CT2
- removed net N$29: R13.1, U3.A1
- removed net N$30: U3.ET1
- removed net N$31: U3.ET2
- removed net N$32: U3.ET3
- removed net N$34: U3.ET4
- removed net N$35: R16.2, U3.A2
- removed net N$36: R19.2, U3.A3
- removed net N$40: R12.1
- removed net N$41: R21.2, R22.2
- removed net N$43: R20.2, U3.A4
- removed net N$44: IC4C.O
- removed net N$45: IC4B.O
- removed net N$46: IC4A.O
- removed net N$50: IC4D.O
- removed net N$51: IC4E.O
- removed net N$52: IC4F.O
- removed net N$67: JP3.2
- removed net N$68: Q2.C
- removed net N$70: JP6.6, R25.1
- removed net N$71: JP4.3, R23.1
- removed net N$72: JP4.4
- removed net N$73: JP5.2
- removed net N$74: JP4.6
- removed net N$75: JP5.3
- removed net N$76: JP6.5, R26.1
- removed net N$77: JP4.14
- removed net N$78: JP4.13
- removed net N$79: JP4.12
- removed net N$80: JP4.11
- removed net N$81: JP6.4, R27.1
- removed net N$82: JP6.3, R28.1
- removed net N$83: JP6.2, R29.1
- removed net N$84: U2.CT3
- removed net N$85: JP7.7, R33.2
- removed net N$86: R24.1
- removed net N$87: JP7.1, R30.2
- removed net N$88: JP7.2
- removed net N$90: JP7.4
- removed net N$92: JP7.6
- removed net N$93: JP7.8
- removed net N$95: JP7.10
- removed net N$97: JP7.12
- removed net VCC_2: JP2.8, JP3.1, R13.2, R16.1, R19.1, R20.1
- new net L-IN1: IC4A.I, R2.2, U1.CT1
- new net L-IN2: IC4B.I, R3.2, U1.CT2
- new net L-IN3: IC4C.I, R5.1, U1.CT3
- new net L-IN4: IC4D.I, R6.1, U1.CT4
- new net L-IN5: IC1A.I, R10.2, U2.CT1
- new net L-IN6: IC1B.I, R11.2, U2.CT2
- new net L-IN7: IC1C.I, R23.2, U2.CT3
- new net L-O1: R1.2, X2-7.K
- new net L-O2: R4.1, X2-6.K
- new net L-O3: R7.1, X2-5.K
- new net L-O4: R8.1, X2-4.K
- new net L-O5: R9.2, X2-3.K
- new net L-O6: R12.1, X2-2.K
- new net L-O7: R24.1, X2-1.K
- new net LED-6: LED6.A, U$1.D48
- new net N$47: Q2.C, X1-2.S
- new net N$56: DS1.VO, R36.1
- new net R-O1: U3.ET1, X3-5.K
- new net R-O2: U3.ET2, X3-4.K
- new net R-O3: U3.ET3, X3-3.K
- new net R-O4: U3.ET4, X3-2.K
- new net VCC-ISO: J2.PWR, JP2.8, R14.1, R15.1, R17.2, R18.2, U$8.IN+, X1-1.S, X2-8.K, X6-1.K
- new net VO-STEP: U$7.S, U$8.OUT+
- net 1A: now also X6-5.K
- net 1B: now also JP2.5, X6-4.K; no longer JP2.3
- net 2A: now also JP2.3, X6-6.K; no longer JP2.5
- net 2B: now also X6-3.K
- net BTN-1: now also R29.1, S5.2, U$1.D34; no longer U$1.A14
- net BTN-2: now also R28.1, S4.2, U$1.D36; no longer U$1.D32
- net BTN-3: now also R27.1, S3.2, U$1.D32; no longer U$1.D34
- net BTN-4: now also R26.1, S2.2, U$1.D3; no longer U$1.D36
- net BTN-5: now also R25.1, S1.2, U$1.D5; no longer U$1.D38
- net BUZ-12V: now also R22.2
- net BUZ-5V: now also R21.2
- net DHT: now also X4-3.S
- net GND: now also DS1.K, DS1.R/!W, DS1.VSS, IC1P.GND, R37.2, R38.2, R39.2, R41.2, R42.2, U$8.OUT-, X4-1.S, X5-4.S; no longer JP4.1, JP4.16, JP4.5, JP5.4, JP8.1, Q2.E
- net GND-ISO: now also J2.GND, J2.GNDBREAK, Q2.E, U$8.IN-, X3-1.K, X6-2.K
- net LCD-D11: now also DS1.DB6, U$1.D10; no longer U$1.A8
- net LCD-D12: now also DS1.DB7, U$1.D12; no longer U$1.A10
- net LCD-D2: now also DS1.RS, U$1.D2; no longer U$1.A0
- net LCD-D3: now also DS1.E, U$1.D4; no longer U$1.A2
- net LCD-D4: now also DS1.DB4, U$1.D6; no longer U$1.A4
- net LCD-D5: now also DS1.DB5, U$1.D8; no longer U$1.A6
- net LED-1: now also LED1.A
- net LED-2: now also LED2.A
- net LED-3: now also LED3.A
- net LED-4: now also LED4.A
- net LED-5: now also LED5.A, U$1.D47; no longer U$1.D48
- net LIM-B1: now also IC4A.O, U$1.D31; no longer U$1.D22
- net LIM-B2: now also IC4B.O, U$1.D30; no longer U$1.D24
- net LIM-B3: now also IC4C.O, U$1.D28; no longer U$1.D26
- net LIM-B4: now also IC4D.O, U$1.D26; no longer U$1.D28
- net LIM-CTR: now also IC1C.O
- net LIM-S1: now also IC1A.O, U$1.D24; no longer U$1.D30
- net LIM-S2: now also IC1B.O, U$1.D22; no longer U$1.D31
- net N$8: now also LED1.C, R30.2; no longer IC5G$1.T1IN
- net N$89: now also LED2.C; no longer JP7.3
- net N$9: now also LED4.C, R33.2; no longer IC5G$1.R1OUT
- net N$91: now also LED3.C; no longer JP7.5
- net N$94: now also LED5.C; no longer JP7.9
- net N$96: now also LED6.C; no longer JP7.11
- net RL-1: now also R13.1, U3.A1
- net RL-2: now also R16.2, U3.A2
- net RL-3: now also R19.2, U$1.D29, U3.A3; no longer U$1.D27
- net RL-4: now also R20.2, U$1.D27, U3.A4; no longer U$1.D29
- net RX-DB9: now also IC5G$1.R1OUT
- net RX-PWR: now also X5-3.S
- net SPDT-1: now also R39.1, U$2.P
- net SPDT-2: now also R37.1, U$3.P
- net SPDT-3: now also R42.1, U$4.P
- net SPDT-4: now also R38.1, U$5.P
- net SPDT-5: now also R41.1, U$6.P
- net TX-DB9: now also IC5G$1.T1IN
- net TX-PWR: now also X5-2.S
- net VCC: now also DS1.A, DS1.VDD, IC1P.VCC, R13.2, R16.1, R19.1, R20.1, R23.1, R36.2, S1.1, S2.1, S3.1, S4.1, S5.1, U$2.S, U$3.S, U$4.S, U$5.S, U$6.S, U$7.P, X4-2.S, X5-1.S; no longer JP4.15, JP4.2, JP5.1, JP6.1, JP8.2, R14.1, R15.1, R17.2, R18.2, R23.2
Other:
- moved on the sheet: C1, C2, C3, C4, C5, IC4A, IC4B, IC4C, IC4D, IC4E, IC4F, IC4P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
